File: listener_hw2/most_listener_v2.kicad_pcb (KiCad board)
At the start: 4 copper layers, 98 x 60 mm, 168 parts, among them J1 1-1394640-1, J2 ANALYSER, J3 I2S, J4 VBAT_IN, J5 FCR684208R, J6 FCR684208T, J7 RCA 75R, J8 LINE L, J9 LINE R, M1 Tang Nano 20K, M2 ESP32-DevKitC-VIE, U1 74LVC1G34, U10 TPS2553DBVR, U11 74LVC1G123, U12 DIR9001, U13 SRC4192, U14 LP5907MFX-3.3, U15 PCM5102A, U16 LP5907MFX-3.3, U17 OPA1678, U18 TPS60403, U2 74LVC1G157, U3 74LVC1G125, U4 74LVC1G123, U5 TPS7B8133DRV, U6 LMR38020F, U7 Si514, U8 LP5907MFX-3.3, U9 74LVC1G79, X1 24.576MHz

Commit message: Listener v2.0: the board after the edit rounds and two reviews of 2026-10-11
The user moved parts in KiCad round by round, each with a sketch, and the copper was re-laid under
every move. Then came two critical reviews, the silk and the fab package. v1.6 (listener_hw/) only
gains one LCSC row in make_fab.py, which v2.0's package shares; v1.6's own package does not change
(it has no 10R).
- The user's moves: L2/D1/D2/F1/C83 and the bottom's C37/FB3/C30/R25/R20, U10's group, R6,
  R50/R51, R11/R12 by U7, U11's C25/R23/C26, the jacks J6..J9 grouped, and three M2.5 mounting
  holes (H1..H3).
- Fewer vias where one side will do: the 5V_SW bus runs on the top, J2's six resistors went to the
  bottom so its lines need no via, J3's hop vias are gone. The router's jogs at pad entries were
  straightened.
- M1 and M2 keep only the pins in use and the corner pins that hold them (gen_listener2.py
  MODULE_FREE_PINS): 12 pads off M1, 25 off M2. The symbols and footprints follow.
- Review 1 (EMC, layout rules, matching, the DAC and its filter), items 1-5, and 7 by the user's
  sketch:
  - R47 10R + C84 10u: 5V_A for the line out (U17's V+, U16, C50, C76, C79);
  - R48 10R + C85 10u: VNEG_A from U18's VNEG_P;
  - R49..R51 33R in BCLK, LRCK and DOUT to the DAC and the ESP32; R52 33R in RX_IN at U3;
  - the main 5V_SW feed to D3, U10 and U18 no longer passes through C76's and U17's pads;
    C43 (100n) stands at U6's VIN;
  - item 7: TX_PRE moved up and RT_CLK took its lane, off the 5.6 mm run at 0.32 mm beside TX_FB.
- The FOT block is the reader v2.0's (JLR-MOST-Reader/reader_hw2): its 19 parts at the reader's
  places by J1's offset, with its copper, and R53 33R after U1 (the reader's R43). RX_BUF goes round
  J1's pins behind its pegs; U3, R52 and C12 sit south-east of J1.
- Review 2, items 1-3:
  - ground vias 0.8-1.35 mm from 15 fast-signal vias;
  - the RX_BUF loop 2.1 mm off J1's pins;
  - the 100n of U13 (C36, C38) and U12 (C34) under the chips on the bottom: U13's 0.6-3.6 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
Parts:
- added C84: 10u, Capacitor_SMD:C_0805_2012Metric, B.Cu at (70.0, 31.1)
- added C85: 10u, Capacitor_SMD:C_0805_2012Metric, B.Cu at (78.4, 44.0)
- added H1: MountingHole_2.7mm_M2.5, MountingHole:MountingHole_2.7mm_M2.5, F.Cu at (53.1, 3.40)
- added H2: MountingHole_2.7mm_M2.5, MountingHole:MountingHole_2.7mm_M2.5, F.Cu at (81.2, 3.25)
- added H3: MountingHole_2.7mm_M2.5, MountingHole:MountingHole_2.7mm_M2.5, F.Cu at (19.3, 56.9)
- added R47: 10, Resistor_SMD:R_0603_1608Metric, B.Cu at (76.1, 34.4)
- added R48: 10, Resistor_SMD:R_0603_1608Metric, B.Cu at (80.9, 43.5)
- added R49: 33, Resistor_SMD:R_0603_1608Metric, B.Cu at (37.3, 46.3)
- added R50: 33, Resistor_SMD:R_0603_1608Metric, B.Cu at (34.4, 46.4)
- added R51: 33, Resistor_SMD:R_0603_1608Metric, B.Cu at (35.2, 42.0)
- added R52: 33, Resistor_SMD:R_0603_1608Metric, B.Cu at (27.4, 24.2)
- added R53: 33, Resistor_SMD:R_0603_1608Metric, B.Cu at (16.2, 18.9)
- C34, C36, C38, R18, R19, R34, R35, R36, R37: moved to B.Cu
- moved U3 17.5 mm to (24.0, 24.0)
- moved C12 15.9 mm to (24.1, 25.9), turned to 180 degrees
- moved U5 13.3 mm to (12.9, 12.4), turned to 180 degrees
- moved C8 13.2 mm to (10.6, 8.79)
- moved C3 13.0 mm to (10.6, 12.2), turned to -90 degrees
- moved C36 12.1 mm to (71.3, 21.8), turned to 0 degrees
- moved U4 9.85 mm to (13.8, 2.30), turned to 180 degrees
- moved C38 9.67 mm to (72.3, 25.4)
- moved FB2 9.55 mm to (13.9, 9.48), turned to -90 degrees
- moved C83 9.39 mm to (16.9, 40.4), turned to 180 degrees
- moved C19 8.42 mm to (15.0, 6.24), turned to 90 degrees
- moved C18 7.62 mm to (16.0, 17.1), turned to 180 degrees
- moved R25 7.59 mm to (10.5, 39.6), turned to 180 degrees
- moved FB1 7.18 mm to (16.2, 15.3), turned to 0 degrees
- moved C43 6.38 mm to (29.0, 18.0), turned to 90 degrees
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Connections:
- C50 pad 1: 5V_SW -> 5V_A
- C75 pad 1: VNEG_A -> VNEG_P
- C76 pad 1: 5V_SW -> 5V_A
- C79 pad 1: 5V_SW -> 5V_A
- M2 pad 21: /I2S_LRCK_F -> /I2S_LRCK_D
- M2 pad 22: /I2S_BCLK_F -> /I2S_BCLK_D
- U1 pad 4: /RX_BUF -> Net-(U1-Y)
- U15 pad 13: /I2S_BCLK_F -> /I2S_BCLK_D
- U15 pad 14: /I2S_DOUT_F -> /I2S_DOUT_D
- U15 pad 15: /I2S_LRCK_F -> /I2S_LRCK_D
- U16 pad 1: 5V_SW -> 5V_A
- U16 pad 3: 5V_SW -> 5V_A
- U17 pad 8: 5V_SW -> 5V_A
- U18 pad 1: VNEG_A -> VNEG_P
- U3 pad 4: /RX_IN -> /RX_IN_U3
Routing:
- net /I2S_LRCK_D: track 0.00 -> 43.4 mm, vias 0 -> 2
- net /I2S_BCLK_F: track 44.9 -> 2.89 mm, vias 1 -> 0
- net /I2S_LRCK_F: track 44.3 -> 2.87 mm, vias 3 -> 0
- net /I2S_BCLK_D: track 0.00 -> 41.1 mm, vias 0 -> 1
- net /I2S_DOUT_D: track 0.00 -> 24.1 mm
- net /I2S_DOUT_F: track 34.7 -> 10.8 mm
- net 3V3_SW: track 93.0 -> 69.7 mm, vias 9 -> 4
- net /RX_IN: track 58.1 -> 38.4 mm
- net 5V_A: track 0.00 -> 16.8 mm
- net 5V_SW: track 220.6 -> 208.6 mm, vias 4 -> 3
- net Net-(J1-TXVCC): track 18.7 -> 8.55 mm, vias 1 -> 0
- net Net-(U12-RXIN): track 89.9 -> 98.7 mm
- net Net-(U2-Y): track 1.70 -> 10.3 mm
- net Net-(J5-VOUT): track 8.32 -> 1.96 mm
- net VNEG_P: track 0.00 -> 4.80 mm
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