File: listener_hw2/most_listener_v2.kicad_sch (KiCad schematic)
At the start: 168 parts, among them J1 1-1394640-1, J2 ANALYSER, J3 I2S, J4 VBAT_IN, J5 FCR684208R, J6 FCR684208T, J7 RCA 75R, J8 LINE L, J9 LINE R, M1 Tang Nano 20K, M2 ESP32-DevKitC-VIE, U1 74LVC1G34, U10 TPS2553DBVR, U11 74LVC1G123, U12 DIR9001, U13 SRC4192, U14 LP5907MFX-3.3, U15 PCM5102A, U16 LP5907MFX-3.3, U17 OPA1678, U18 TPS60403, U2 74LVC1G157, U3 74LVC1G125, U4 74LVC1G123, U5 TPS7B8133DRV, U6 LMR38020F, U7 Si514, U8 LP5907MFX-3.3, U9 74LVC1G79, X1 24.576MHz

Commit message: Listener v2.0: the board after the edit rounds and two reviews of 2026-10-11
The user moved parts in KiCad round by round, each with a sketch, and the copper was re-laid under
every move. Then came two critical reviews, the silk and the fab package. v1.6 (listener_hw/) only
gains one LCSC row in make_fab.py, which v2.0's package shares; v1.6's own package does not change
(it has no 10R).
- The user's moves: L2/D1/D2/F1/C83 and the bottom's C37/FB3/C30/R25/R20, U10's group, R6,
  R50/R51, R11/R12 by U7, U11's C25/R23/C26, the jacks J6..J9 grouped, and three M2.5 mounting
  holes (H1..H3).
- Fewer vias where one side will do: the 5V_SW bus runs on the top, J2's six resistors went to the
  bottom so its lines need no via, J3's hop vias are gone. The router's jogs at pad entries were
  straightened.
- M1 and M2 keep only the pins in use and the corner pins that hold them (gen_listener2.py
  MODULE_FREE_PINS): 12 pads off M1, 25 off M2. The symbols and footprints follow.
- Review 1 (EMC, layout rules, matching, the DAC and its filter), items 1-5, and 7 by the user's
  sketch:
  - R47 10R + C84 10u: 5V_A for the line out (U17's V+, U16, C50, C76, C79);
  - R48 10R + C85 10u: VNEG_A from U18's VNEG_P;
  - R49..R51 33R in BCLK, LRCK and DOUT to the DAC and the ESP32; R52 33R in RX_IN at U3;
  - the main 5V_SW feed to D3, U10 and U18 no longer passes through C76's and U17's pads;
    C43 (100n) stands at U6's VIN;
  - item 7: TX_PRE moved up and RT_CLK took its lane, off the 5.6 mm run at 0.32 mm beside TX_FB.
- The FOT block is the reader v2.0's (JLR-MOST-Reader/reader_hw2): its 19 parts at the reader's
  places by J1's offset, with its copper, and R53 33R after U1 (the reader's R43). RX_BUF goes round
  J1's pins behind its pegs; U3, R52 and C12 sit south-east of J1.
- Review 2, items 1-3:
  - ground vias 0.8-1.35 mm from 15 fast-signal vias;
  - the RX_BUF loop 2.1 mm off J1's pins;
  - the 100n of U13 (C36, C38) and U12 (C34) under the chips on the bottom: U13's 0.6-3.6 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
Parts:
- added C84, C85: 10u, Capacitor_SMD:C_0805_2012Metric, symbol Device:C
- added R47, R48: 10, Resistor_SMD:R_0603_1608Metric, symbol Device:R
- added R49, R50, R51, R52, R53: 33, Resistor_SMD:R_0603_1608Metric, symbol Device:R
Connections:
- net 5V_SW: now also R47.1; no longer C50.1, C76.1, C79.1, U16.1 (IN), U16.3 (EN), U17.8 (V+)
- net GND: now also C84.2, C85.2
- net I2S_BCLK_F: now also R49.1; no longer M2.22 (IO22), U15.13 (BCK)
- net I2S_DOUT_F: now also R51.1; no longer U15.14 (DIN)
- net I2S_LRCK_F: now also R50.1; no longer M2.21 (IO23), U15.15 (LRCK)
- net RX_BUF: now also R53.2; no longer U1.4 (Y)
- net RX_IN: now also R52.2; no longer U3.4 (Y)
- net VNEG_A: now also C85.1, R48.2; no longer C75.1, U18.1 (OUT)
- new net: R53.1, U1.4 (Y)
- new net 5V_A: C50.1, C76.1, C79.1, C84.1, R47.2, U16.1 (IN), U16.3 (EN), U17.8 (V+)
- new net I2S_BCLK_D: M2.22 (IO22), R49.2, U15.13 (BCK)
- new net I2S_DOUT_D: R51.2, U15.14 (DIN)
- new net I2S_LRCK_D: M2.21 (IO23), R50.2, U15.15 (LRCK)
- new net RX_IN_U3: R52.1, U3.4 (Y)
- new net VNEG_P: C75.1, R48.1, U18.1 (OUT)
- no-connect marks 58 -> 21
Other:
- note added: "12. v2.0: ФІЛЬТРИ ЖИВЛЕННЯ U17, УЗГОДЖЕННЯ I2S ДО ЦАП І RX_IN"
- note added: "R49-R51: 33 Ом біля FPGA на гілці I2S до ЦАП і ESP32 (BCLK, LRCK, DOUT: 35-45 мм, кілька навантажень; PCM5102A бере такт з BCLK). J3 має свої R39-R41."
- note added: "R52: 33 Ом на виході U3 (RX_IN до FPGA, близько 60 мм)."
- note added: "R53: 33 Ом на виході U1 (RX_BUF до U2, U3, U4; через U2 і R2 - TX кільця), як R43 у рідері v2.0; стоїть у блоці 3."
- note added: "RC 10 Ом / 10 мкФ: зріз 1.6 кГц, на 250 кГц (насос) і на частоті перетворювача близько 45 дБ; спад на R47 до 0.2 В (U17 + U16 з ЦАП), на R48 близько 50 мВ. Бусина з 10 мкФ дала б резонанс на десятках кГц."
- note added: "U17 (OPA1678) більше не живиться прямо від шин: V+ = 5V_A (5V_SW через R47 10 Ом, C84 10 мкФ; від 5V_A живиться й U16, LDO ЦАП), V- = VNEG_A (VNEG_P насоса U18 через R48 10 Ом, C85 10 мкФ)."

Commit message: sheets: block titles and notes in English, for v1.6 and v2.0
The sheets' eleven block titles and their notes were Ukrainian. They are now English in
gen_listener.py, and v2.0's block 12 in gen_listener2.py. Both sheets were generated anew, as
were the schematic PDFs in both fab packages and the kit's copy of v2.0's.

The notes keep their places. English runs wider in KiCad's font, so ten notes were reworded
until each stood no wider than its Ukrainian original or than its frame. A few original
notes already ran past their frames, and those stay as wide as they were.

ERC passes on both sheets. tools/check_v2_circuit.py: 168/168 parts, 125/125 nets, PASS.
Both fab packages differ only in their schematic PDF. make_kit.py --check passes.

Co-Authored-By: Claude Opus 5.5 <noreply@anthropic.com>
Other:
- note added: "(R6 x C9). The ring asleep"
- note added: "-> LOCK = 0 -> bypass."
- note added: "-> TX_SEL = 0: bypass."
- note added: "-> WAKE = 0 -> U6 off,"
- note added: "1. POWER J4 battery -> 3V3_AON (always) and 5V_SW (on WAKE) -> 5V_HOST (M2)"
- note added: "10. TEST POINTS (bench)"
- note added: "11. LINE OUT J3's stereo -> U15 PCM5102A -> J8 L, J9 R (RCA, 2.1 Vrms)"
- note added: "12. v2.0: U17'S SUPPLY FILTERS, I2S TERMINATION TO THE DAC, RX_IN"
- note added: "2. WAKE-UP (U4) AND THE BYPASS WATCHDOG (U11)"
- note added: "3. THE RING J1 = MOST in and out (both fibres); regeneration, always powered"
- note added: "3V3_AON (U5) always: FOT, U1, U2, U4, U11. Parked (the ring asleep) up to ~60 uA in all: the FOT asleep <= 25, logic, LDO 2.7."
- note added: "4. FPGA ISOLATION, TX FLIP-FLOP"
- note added: "5V_HOST (U10): M2's supply (ESP32), limit ~1 A (R22 24k9): the module's radio draws peaks over 0.5 A; 5 V from the module's USB does not flow back into 5V_SW."
- note added: "5V_HOST -> 5V; the module's USB through its own diode."
- note added: "5V_SW (U6 LMR38020, 80 V, 400 kHz) on WAKE: the FPGA module, U14 (3V3_DA, block 9). VOUT 5.31 V. C44/C45 + L2 22 uH: harness ringing damped, 400 kHz kept out."
- note added: "6. THE REGENERATION CLOCK Si514 = 1024 x the ring's FS (45.16 / 49.15 MHz), steered by the FPGA"
- note added: "7. OUTPUTS J2: analyser (MCLK, 2 x TDM8, UART_TX); J3: stereo I2S for a DAC / DSP"
- note added: "8. HOST M2 = ESP32-DevKitC-VIE"
- note added: "9. DIGITAL AUDIO J5 TOSLINK IN -> U12 DIR9001 -> U13 SRC4192 -> I2S_DIN2_F; SPDIF_F -> J6 TOSLINK OUT and J7 coax"
- note added: "At start-up, centring (FCAL, up to 10 ms): the Si514's output is high-impedance then, R14 and R17 hold the lines at 0. U8: its own LDO from 5V_SW."
- note added: "Bench probe points: the 3V3_AON and 5V_SW rails, ground. None on the ring's lines: a stub on their edges"
- note added: "C36/C37 U13 VDD; C38 U13 VIO; C39 X1: by the pins."
- note added: "CLK+ -> FPGA (clk_r = 1024 Fs) and through R15 to U9: the TX edges sit on the Si514's clock, not on the FPGA's output. CLK- is not needed."
- note added: "CLK_1024 (Si514) -> 77 (GCLKT_1). TX_FB -> 25 through IDES8 (1.26 ns); it takes the pair, so 26 is not connected."
- note added: "D3: the USB and 5V_SW are never joined; U6 gives 5.3 V, the module gets ~5.0 V."
- note added: "FB1/FB2 + 100n + 10u: RX and TX separately."
- note added: "IO13 <- OPT_ERR, IO27 <- OPT_NPCM (U12, block 9; v1.3)."
- note added: "Its input is the same stereo as J3's. XSMT = LOCK: the DAC is muted while the ring is not locked and before the FPGA is configured (R8); it ramps over 104 samples."
- note added: "J2 SD0/SD1: the frame's bytes 0..31 / 32..63, a TDM frame = a MOST frame."
- note added: "J2 UART_TX: the raw control blocks (the same M2 reads)."
- note added: "J2 and J3 take no input: the one host is M2 (block 8)."
- note added: "J3: I2S, BCLK 64 Fs, 32-bit slots, 24 bits with the head unit's controls applied; the same on S/PDIF, J6, J7 (block 9)."
- note added: "J4 Molex Micro-Fit 3.0 right-angle 43650-0200 on the left edge under J1 (mating 43645-0200, contacts 43030), latched, 5 A. Protection: F1 2 A slow-blow; D2 SMBJ36A before D1: silent at 35 V (ISO 16750-2 B), clamps ISO 7637-2 pulses to ~50 V."
- note added: "J5 TOSLINK IN -> R25 -> U12 DIR9001: its PLL recovers the clock from the signal, output I2S 24 bit (FMT1 FMT0 = HH), CKSEL = L. XTI to ground: no crystal needed."
- note added: "M2: ESP32-DevKitC-VIE (WROVER-IE): 8 MB PSRAM,"
- note added: "MCLK on J2 and J3 from separate FPGA pins, no branch."
- note added: "OPT_ERR (U12 ERROR) -> M2 IO13: 1 = no TOSLINK signal or a parity error; OPT_NPCM (U12 AUDIO) -> M2 IO27: 1 = not PCM (the DIR9001 does not mute AC-3/DTS); the host then does not inject. Source: command 02, bit M[2]."
- note added: "On the board each capacitor of the row stands by its pin: C52, C53 CPVDD; C54, C55 AVDD; C56 DVDD."
- note added: "Output 2.1 Vrms ground-referenced, no coupling caps. U17: buffer with a 2nd-order Sallen-Key low-pass (Butterworth, 60 kHz), C0G; then 100 ohm + 2.2 nF, D5, D6 (ESD) at the RCA."
- note added: "Pins 1..20 / 21..40 top to bottom, from the USB-C; name = the GW2AR pin + what the module has on it (data sheet v1.3)."
- note added: "Pins 2 x 1x19, 2.54 pitch, the rows 25.40 mm apart."
- note added: "Q -> U2 (TX_REGEN) and into the FPGA (TX_FB)."
- note added: "R18..R21, R34..R41 (33 ohm): each by its FPGA pin (source termination); R38..R41 under M2."
- note added: "R49-R51: 33 ohm at the FPGA on the I2S branch to the DAC and ESP32 (BCLK, LRCK, DOUT: 35-45 mm, many loads; the DAC clocks off BCLK). J3: R39-R41."
- note added: "R52: 33 ohm at U3's output (RX_IN to the FPGA, about 60 mm)."
- note added: "R53: 33 ohm at U1's output (RX_BUF to U2, U3, U4; through U2 and R2 the ring's TX), as R43 in the reader v2.0; drawn in block 3."
- note added: "R7: RXD held at 0 while the receiver sleeps."
- note added: "R8: FPGA not configured"
- note added: "RC 10 ohm / 10 uF: corner 1.6 kHz, ~45 dB at 250 kHz (the pump) and the buck's frequency; R47 drops up to 0.2 V (U17 + U16 with the DAC), R48 ~50 mV. A bead with 10 uF would ring at tens of kHz."
- note added: "S = 1 (LOCK and TX edges, U11): TX = the regenerated signal from the FPGA. The network does not see us."
- note added: "S = TX_SEL = 0: FPGA off, not locked, or TX stuck -> straight through RX -> TX."
- note added: "S/PDIF OUT: SPDIF_F (FPGA 42) -> R28 -> J6 FCR684208T; R26/R27: 0.5 V into 75 ohm, 75 ohm out; C29 blocks DC -> J7 RCA. The same stream as on J3."
- note added: "STATUS's polarity"
- note added: "TX stuck (clock, U9, FPGA)"
- note added: "The FPGA finds the Si514's I2C address itself (it tries 0x08..0x77) and steers M (dpll.v): TX_FB's delay against RX_IN within 1.26 ns, steps of 0.026 ppb."
- note added: "The ring and the Si514 on the LCD pins only (an empty connector): LOCK on 31, S/PDIF on 42. HSPI, 54..56 (the module amplifier's inputs; PA_EN = 51 keeps it off), EDID 52/53: UART, MCLK, I2S, SD1, DIN2."
- note added: "U11: TX_SEL = 1 only"
- note added: "U13 SRC4192: both ports slave (MODE = 000); input I2S 24 bit (IFMT = 001) from U12; output I2S 24 bit (OFMT = 01, OWL = 00) on the FPGA's clocks (their own copies of BCLK, LRCK: SRC_BCLK_F, SRC_LRCK_F) -> I2S_DIN2_F."
- note added: "U14 LP5907: 3V3_DA (250 mA) for block 9 from 5V_SW, not from the module's LDO. J7 pad 3 (the thin pin off the axis): BKL's drawing gives it no function; measure on a sample."
- note added: "U15 PCM5102A, hardware mode: FMT = 0 (I2S), FLT = 0 (normal latency), DEMP = 0. SCK to ground: the PLL takes its clock from BCK (3 wires, BCK = 64 Fs)."
- note added: "U16 LP5907: 3V3_DAC from 5V_SW. Its output takes at most 10 uF, so AVDD 4.7 uF and CPVDD 2.2 uF instead of fig. 33's 10 uF."
- note added: "U17 (OPA1678) no longer runs straight off the rails: V+ = 5V_A (5V_SW via R47 10 ohm, C84 10 uF; it feeds U16, the DAC's LDO, too), V- = VNEG_A (U18's VNEG_P via R48 10 ohm, C85 10 uF)."
- note added: "U17 on +5V_SW and VNEG_A (-5.2 V, U18 TPS60403): output to the rails, input to V-, so +-3 V of signal fits with margin. J8, J9 pad 3: as J7's, measure a sample."
- note added: "U3, U9 on 3V3_SW: when the FPGA"
- note added: "U4: every RX edge"
- note added: "U7 Si514: any off-the-shelf 3.3 V CMOS one - after 514 in the part number the letter C, M or N; package 3.2x5 or 2.5x3.2 (the letter before AG: B or C), both fit one land pattern."
- note added: "U9: the TX edges on the Si514's clock (RT_CLK)."
- note added: "UART 3 Mbaud: IO4 <- UART_TX, IO15 -> R20 -> UART_RX."
- note added: "X1 24.576 MHz: the reference clock of the SRC4192's rate estimator (RCKI), asynchronous to both ports. RST_AIN: R30/C40 = 10 ms, once X1 runs (the SRC4192 has no POR)."
- note added: "an IPEX antenna (external, 2.4 GHz), -40...85 °C."
- note added: "fibre FROM the previous node -> RX"
- note added: "fibre TO the next node <- TX"
- note added: "has found the rate ratio."
- note added: "is off, they (Ioff) do not load the lines."
- note added: "longer is not MOST)."
- note added: "need not be known."
- note added: "on TX_REGEN (R23 x C25"
- note added: "restarts ~0.1 s"
- note added: "the FPGA unpowered."
- note added: "v1.2: J2's and J3's pin order follows their pins on M1's right row; the tracks do not cross."
- note added: "v1.2: lines to the right leave the right row as J2, J3, DAC, host; U13's (SRC_BCLK, SRC_LRCK, DIN2) the left row, over M1."
- note added: "v1.2: the links to the FPGA on the row facing M1."
- note added: "v1.3: RDY -> MUTE - silent until the SRC4192"
- note added: "while LOCK = 1 and edges"
- note added: "would hurt. RX_BUF at U1 pin 4, TX_SEL at U2 pin 6, TX_REGEN and RT_CLK at U9 and at M1 (TX_FB)."
- note added: "~10 us; TX without edges"
- note removed: "(R6 x C9). Кільце спить"
- note removed: "-> LOCK = 0 -> обхід."
- note removed: "-> TX_SEL = 0: обхід."
- note removed: "-> WAKE = 0 -> U6 вимк.,"
- note removed: "1. ЖИВЛЕННЯ J4 акумулятор -> 3V3_AON (завжди) і 5V_SW (за WAKE) -> 5V_HOST (M2)"
- note removed: "10. ТЕСТОВІ ТОЧКИ (стенд)"
- note removed: "11. ЛІНІЙНИЙ ВИХІД стерео J3 -> U15 PCM5102A -> J8 L, J9 R (RCA, 2.1 Вrms)"
- note removed: "12. v2.0: ФІЛЬТРИ ЖИВЛЕННЯ U17, УЗГОДЖЕННЯ I2S ДО ЦАП І RX_IN"
- note removed: "2. ПРОБУДЖЕННЯ (U4) І СТОРОЖ ОБХОДУ (U11)"
- note removed: "3. КІЛЬЦЕ J1 = вхід і вихід MOST (обидва волокна); ретрансляція, завжди живлено"
- note removed: "3V3_AON (U5) завжди: FOT, U1, U2, U4, U11. На стоянці (кільце спить) разом до ~60 мкА: FOT у сні <= 25, логіка, LDO 2.7."
- note removed: "4. РОЗВ'ЯЗКА FPGA, ТРИГЕР TX"
- note removed: "5V_HOST (U10): живлення M2 (ESP32), межа ~1 А (R22 24k9): радіо модуля бере піки понад 0.5 А; 5 В з USB модуля назад у 5V_SW не проходять."
- note removed: "5V_HOST -> 5V; USB модуля - через його діод."
- note removed: "5V_SW (U6 LMR38020, 80 В, 400 кГц) вмикає WAKE: модуль FPGA і U14 (3V3_DA, блок 9). VOUT 5.31 В. C44/C45 + L2 22 мкГн: дзвін джгута і 400 кГц не в джгут."
- note removed: "6. ТАКТ ПЕРЕГЕНЕРАЦІЇ Si514 = 1024 x FS кільця (45.16 / 49.15 МГц), крутить FPGA"
- note removed: "7. ВИХОДИ J2: аналізатор (MCLK, 2 x TDM8, UART_TX); J3: стерео I2S для ЦАП / DSP"
- note removed: "8. ХОСТ M2 = ESP32-DevKitC-VIE"
- note removed: "9. ЦИФРОВЕ АУДІО J5 TOSLINK IN -> U12 DIR9001 -> U13 SRC4192 -> I2S_DIN2_F; SPDIF_F -> J6 TOSLINK OUT і J7 коаксіал"
- note removed: "C36/C37 U13 VDD; C38 U13 VIO; C39 X1: біля виводів."
- note removed: "CLK+ -> FPGA (clk_r = 1024 Fs) і через R15 на U9: фронти TX стоять на такті Si514, а не на виході FPGA. CLK- не потрібен."
- note removed: "CLK_1024 (Si514) -> 77 (GCLKT_1). TX_FB -> 25 через IDES8 (1.26 нс); він займає пару, тому 26 не підключено."
- note removed: "D3: USB і 5V_SW разом не з'єднуються; U6 дає 5.3 В, на модулі ~5.0 В."
- note removed: "FB1/FB2 + 100n + 10u: RX і TX окремо."
- note removed: "FPGA без живлення."
- note removed: "FPGA сама знаходить I2C адресу Si514 (перебирає 0x08..0x77) і крутить M (dpll.v): затримка TX_FB відносно RX_IN до 1.26 нс, крок 0.026 ppb."
- note removed: "IO13 <- OPT_ERR, IO27 <- OPT_NPCM (U12, блок 9; v1.3)."
- note removed: "J2 SD0/SD1: байти кадру 0..31 / 32..63, кадр TDM = кадр MOST."
- note removed: "J2 UART_TX: сирі керувальні блоки (ті самі, що читає M2)."
- note removed: "J3: I2S, BCLK 64 Fs, слоти 32 біт, 24 біт з регулюваннями ГУ; те саме S/PDIF - J6, J7 (блок 9)."
- note removed: "J4 Molex Micro-Fit 3.0 кутовий 43650-0200 на лівому краю під J1 (відповідна частина 43645-0200, контакти 43030), із защіпкою, 5 А. Захист: F1 2 А інерційний; D2 SMBJ36A перед D1: мовчить при 35 В (ISO 16750-2 B), імпульси ISO 7637-2 тисне до ~50 В."
- note removed: "J5 TOSLINK IN -> R25 -> U12 DIR9001: PLL відновлює такт із сигналу, вихід I2S 24 біт (FMT1 FMT0 = HH), CKSEL = L. XTI на землю: кварц не потрібен."
- note removed: "M2: ESP32-DevKitC-VIE (WROVER-IE): 8 МБ PSRAM,"
- note removed: "MCLK на J2 і J3 - з окремих виводів FPGA, без відгалуження."
- note removed: "OPT_ERR (U12 ERROR) -> M2 IO13: 1 = TOSLINK без сигналу або помилка парності; OPT_NPCM (U12 AUDIO) -> M2 IO27: 1 = не PCM (AC-3/DTS DIR9001 не глушить); хост тоді не інжектує. Джерело: команда 02, біт M[2]."
- note removed: "Q -> U2 (TX_REGEN) і в FPGA (TX_FB)."
- note removed: "R18..R21, R34..R41 (33 Ом): кожен біля свого виводу FPGA (узгодження джерела); R38..R41 - під M2."
- note removed: "R49-R51: 33 Ом біля FPGA на гілці I2S до ЦАП і ESP32 (BCLK, LRCK, DOUT: 35-45 мм, кілька навантажень; PCM5102A бере такт з BCLK). J3 має свої R39-R41."
- note removed: "R52: 33 Ом на виході U3 (RX_IN до FPGA, близько 60 мм)."
- note removed: "R53: 33 Ом на виході U1 (RX_BUF до U2, U3, U4; через U2 і R2 - TX кільця), як R43 у рідері v2.0; стоїть у блоці 3."
- note removed: "R7: RXD у 0, коли приймач спить."
- note removed: "R8: FPGA не завантажена"
- note removed: "RC 10 Ом / 10 мкФ: зріз 1.6 кГц, на 250 кГц (насос) і на частоті перетворювача близько 45 дБ; спад на R47 до 0.2 В (U17 + U16 з ЦАП), на R48 близько 50 мВ. Бусина з 10 мкФ дала б резонанс на десятках кГц."
- note removed: "S = 1 (LOCK і фронти TX, U11): TX = перегенерований сигнал з FPGA. Мережа нас не бачить."
- note removed: "S = TX_SEL = 0: FPGA вимкнена, без захоплення або TX став -> прямий прохід RX -> TX."
- note removed: "S/PDIF OUT: SPDIF_F (FPGA 42) -> R28 -> J6 FCR684208T; R26/R27: 0.5 В на 75 Ом, вихідний опір 75 Ом; C29 без постійної -> J7 RCA. Той самий потік, що й на J3."
- note removed: "TX став (такт, U9, FPGA)"
- note removed: "TX_REGEN є (R23 x C25"
- note removed: "U11: TX_SEL = 1, лише"
- note removed: "U13 SRC4192: обидва порти slave (MODE = 000); вхід I2S 24 біт (IFMT = 001) від U12; вихід I2S 24 біт (OFMT = 01, OWL = 00) на тактах FPGA (власні копії BCLK, LRCK: SRC_BCLK_F, SRC_LRCK_F) -> I2S_DIN2_F."
- note removed: "U14 LP5907: 3V3_DA (250 мА) для блоку 9 від 5V_SW, не з LDO модуля. J7 пад 3 (тонкий штир поза віссю): функції в кресленні BKL нема, зміряти на зразку."
- note removed: "U15 PCM5102A, апаратний режим: FMT = 0 (I2S), FLT = 0 (звичайна затримка), DEMP = 0. SCK на землі: PLL бере такт з BCK (3 проводи, BCK = 64 Fs)."
- note removed: "U16 LP5907: 3V3_DAC від 5V_SW. Ємність на його виході - до 10 мкФ, тому AVDD 4.7 мкФ і CPVDD 2.2 мкФ замість 10 мкФ з рис. 33."
- note removed: "U17 (OPA1678) більше не живиться прямо від шин: V+ = 5V_A (5V_SW через R47 10 Ом, C84 10 мкФ; від 5V_A живиться й U16, LDO ЦАП), V- = VNEG_A (VNEG_P насоса U18 через R48 10 Ом, C85 10 мкФ)."
- note removed: "U17 живиться від +5V_SW і VNEG_A (-5.2 В, U18 TPS60403): вихід до шин, вхід до V-, тож +-3 В сигналу проходять з запасом. J8, J9 пад 3: як у J7, зміряти на зразку."
- note removed: "U3, U9 від 3V3_SW: коли FPGA"
- note removed: "U4: кожен фронт RX"
- note removed: "U7 Si514: будь-який з полиці з 3.3 В CMOS - у номері після 514 літера C, M або N; корпус 3.2x5 або 2.5x3.2 (літера перед AG: B або C), обидва сідають на одне посадкове місце."
- note removed: "U9: фронти TX на такті Si514 (RT_CLK)."
- note removed: "UART 3 Мбод: IO4 <- UART_TX, IO15 -> R20 -> UART_RX."
- note removed: "X1 24.576 МГц: опорний такт оцінювача швидкості SRC4192 (RCKI), асинхронний до обох портів. RST_AIN: R30/C40 = 10 мс, коли X1 уже іде (SRC4192 без POR)."
- note removed: "v1.2: зв'язки з FPGA - на ряду, що дивиться на M1."
- note removed: "v1.2: лінії праворуч - з правого ряду в порядку J2, J3, ЦАП, хост; U13 (SRC_BCLK, SRC_LRCK, DIN2) - з лівого ряду понад модулем."
- note removed: "v1.2: порядок контактів J2 і J3 - як їхні виводи на правому ряду M1, доріжки без перехрещень."
- note removed: "v1.3: RDY -> MUTE - тиша, поки SRC4192"
- note removed: "~10 мкс; TX без фронтів"
- note removed: "Вихід 2.1 Вrms відносно землі, без розділових конденсаторів. U17: повторювач з ФНЧ Саллена-Кі 2-го порядку (Баттерворт, 60 кГц), C0G; далі 100 Ом + 2.2 нФ і D5, D6 (ESD) на RCA."
- note removed: "Входів на J2 і J3 немає: хост один - M2 (блок 8)."
- note removed: "Вхід - те саме стерео, що на J3. XSMT = LOCK: без захоплення кільця і до конфігурації FPGA (R8) ЦАП приглушений; спад і підйом за 104 відліки."
- note removed: "Гнізда 2 x 1x19, крок 2.54, між рядами 25.40 мм."
- note removed: "Контакти 1..20 / 21..40 згори вниз, від USB-C; назва = вивід GW2AR + що на ньому на платі (datasheet v1.3)."
- note removed: "Кільце і Si514 - лише на виводах LCD (порожній роз'єм): LOCK на 31, S/PDIF на 42. HSPI, 54..56 (входи підсилювача модуля; PA_EN = 51 тримає його вимкненим), EDID 52/53: UART, MCLK, I2S, SD1, DIN2."
- note removed: "На платі кожен конденсатор ряду стоїть біля свого виводу: C52, C53 - CPVDD; C54, C55 - AVDD; C56 - DVDD."
- note removed: "На старті центрування (FCAL, до 10 мс): вихід Si514 тоді у високому імпедансі, R14 і R17 тримають лінії в 0. U8: окремий LDO з 5V_SW."
- note removed: "Полярність STATUS"
- note removed: "Під щуп на стенді: шини 3V3_AON і 5V_SW, земля. Лінії кільця без точок: відвід на їхніх фронтах"
- note removed: "антена IPEX (виносна, 2.4 ГГц), -40...85 °C."
- note removed: "вимкнена, вони (Ioff) не вантажать лінії."
- note removed: "волокно ВІД попереднього вузла -> RX"
- note removed: "волокно ДО наступного вузла <- TX"
- note removed: "довше - не MOST)."
- note removed: "зайвий. RX_BUF - на виводі 4 U1, TX_SEL - на виводі 6 U2, TX_REGEN і RT_CLK - на U9 і на M1 (TX_FB)."
- note removed: "знати не треба."
- note removed: "не визначив співвідношення частот."
- note removed: "перезапускає ~0.1 с"
- note removed: "поки LOCK = 1 і фронти"
